File: hardware/warp-energy-manager.kicad_pcb (KiCad board)
At the start: 4 copper layers, 68 x 87 mm, 105 parts, among them J101 Boot, J102 DM3CS, P101 CON-SENSOR2, P102 Relay, P103 L+N, P104 OUT, P105 INPUT, P106 DNP, P110 MODBUS, P111 Debug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

Commit message: fix routing
Routing:
- net SD-CDS: track 44.7 -> 45.8 mm
